File: PCB/Quantum-MINI.kicad_pcb (KiCad board)
At the start: 2 copper layers, 250.6 x 155.2 mm, 85 parts, among them J2 JTAG_TC2030, J3 USB_A, J4 Conn_01x06, SW1 Boot, SW10 MX_SW_HS, SW11 MX_SW_solder, SW12 MX_SW_solder, SW13 MX_SW_HS, SW14 MX_SW_solder, SW15 MX_SW_HS, SW16 MX_SW_solder, SW17 MX_SW_HS, SW18 MX_SW_HS, SW19 MX_SW_solder, SW2 MX_SW_HS, SW20 MX_SW_HS, SW21 MX_SW_solder, SW22 MX_SW_solder, SW23 MX_SW_HS, SW24 MX_SW_HS, SW25 MX_SW_solder, SW26 MX_SW_HS, SW27 MX_SW_solder, SW28 MX_SW_HS, SW29 MX_SW_solder, SW3 MX_SW_solder, SW30 MX_SW_solder, SW31 MX_SW_HS, SW32 MX_SW_HS, SW33 MX_SW_solder, SW34 MX_SW_solder, SW35 MX_SW_HS, SW36 MX_SW_HS, SW37 MX_SW_solder, SW38 MX_SW_solder, SW39 MX_SW_HS, SW4 MX_SW_HS, SW40 MX_SW_HS, SW41 MX_SW_solder, SW42 SW_SPDT, SW5 MX_SW_solder, SW6 MX_SW_solder, SW7 MX_SW_HS, SW8 MX_SW_solder, SW9 MX_SW_HS, U1 XC6206, U3 RP2040, U4 W25Q128JVS, U5 USBLC6-2SC6, U6 W25Q128JVS, Y1 12MHz

Commit message: Uploaded latest changes
Parts:
- added J1: Conn_01x04, DevLibrary:SH1107, F.Cu at (148.5, 91.1)
- SW42: footprint Button_Switch_SMD:SW_SPDT_PCM12 -> Button_Switch_THT:SW_CuK_OS102011MA1QN1_SPDT_Angled
- moved R13 160.9 mm to (125.9, -0.28)
- moved R10 146.8 mm to (122.6, 24.0)
- moved SW1 146.8 mm to (127.8, 25.8)
- moved U6 143.3 mm to (117.5, 27.8), turned to -90 degrees
- moved C19 141.2 mm to (121.0, 29.6)
- moved U4 137.6 mm to (109.8, 29.8), turned to 0 degrees
- moved SW42 19.3 mm to (105.0, 24.2)
- moved J4 2.30 mm to (154.8, 57.3)
Connections:
- U3 pad 11: unconnected-(U3-GPIO8-Pad11) -> SDA
- U3 pad 12: unconnected-(U3-GPIO9-Pad12) -> SCL
Routing:
- net Net-(J3-Shield): track 18.2 -> 31.3 mm
- net SD3: track 10.5 -> 2.47 mm
- net QSPI_CLK: track 9.31 -> 2.43 mm
- net +3V3: track 65.7 -> 60.0 mm
- net SD0: track 7.55 -> 2.20 mm
- net CS: track 6.52 -> 2.24 mm
- net SD2: track 7.12 -> 3.22 mm
- net SD1: track 6.63 -> 2.73 mm
- net GND: track 49.1 -> 51.6 mm, vias 18 -> 19
- net (no net): vias 1 -> 0
